Commit message: Added extruder + first joint

File: move_printer/urdf/printer.urdf (robot description, URDF)
Before this commit: robot printer, 1 links, 0 joints
Links:
- added link extruder_link; visual cylinder length=${extruder_length} radius=${extruder_radius}
Joints:
- added joint joint1: type prismatic, parent base_link, child extruder_link, origin xyz=0 0 0.35 rpy=0 0 0, limit lower=${-plate_length/2} upper=${plate_length/2} effort=1000.0 velocity=0.1

Commit message: Added 3 axis extruder in urdf

File: move_printer/urdf/printer.urdf (robot description, URDF)
Before this commit: robot printer, 2 links, 1 joints
Links:
- added link extruder_link_virt1
- added link extruder_link_virt2
Joints:
- added joint joint2: type prismatic, parent extruder_link_virt1, child extruder_link_virt2, origin xyz=0 0 0 rpy=0 0 0, axis 0 1 0, limit lower=${-plate_length/2} upper=${plate_length/2} effort=1000.0 velocity=0.1
- added joint joint3: type prismatic, parent extruder_link_virt2, child extruder_link, origin xyz=0 0 0.35 rpy=0 0 0, axis 0 0 1, limit lower=${-extruder_max_height} upper=0 effort=1000.0 velocity=0.1
- joint joint1: axis (none) -> 1 0 0; child extruder_link -> extruder_link_virt1; origin xyz=0 0 0.35 rpy=0 0 0 -> xyz=0 0 0 rpy=0 0 0
